File: hardware/flight_controller_pcb/qcopter_fc_carrier.kicad_pcb (KiCad board)
At the start: 4 copper layers, 95 x 85 mm, 22 parts, among them J1 Pico 2 pins 1-20, J10 CC1101 B SPI/GDO (3V3), J11 ESC FL signal/GND, J12 ESC FR signal/GND, J13 ESC RR signal/GND, J14 ESC RL signal/GND, J15 AUX UART 3V3/GND/TX/RX, J2 Pico 2 pins 40-21, J3 3S input (low-current branch), J4 External 5 V buck module: VIN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, J5 MPU6050 I2C, J6 BMP280 I2C, J7 HMC5883L I2C, J8 LoRa SPI/DIO (3V3), J9 CC1101 A SPI/GDO (3V3)

Commit message: feat: add battery estimation and safety interfaces
Parts:
- added C2: 100n current ADC filter, Capacitor_SMD:C_0805_2012Metric, F.Cu at (78.0, 12.0)
- added J16: 3V3 current sensor output only, Connector_PinHeader_2.54mm:PinHeader_1x03_P2.54mm_Vertical, F.Cu at (87.0, 12.0)
- added J17: External 3S monitor I2C/ALERT (not power path), Connector_PinHeader_2.54mm:PinHeader_1x05_P2.54mm_Vertical, F.Cu at (78.0, 68.0)
- added R3: 1k current ADC series filter, Resistor_SMD:R_0805_2012Metric, F.Cu at (72.0, 12.0)
Connections:
- J2 pad 7: GND -> BMS_ALERT
- J2 pad 8: GPIO_SPARE_28 -> GND
- J2 pad 9: GPIO_SPARE_27 -> IBAT_ADC
Other:
- board text added: "CELL MONITOR I2C"
- board text added: "CURRENT SIGNAL"
