File: hardware/home-etched-fc/esp32_home_etch.kicad_sch (KiCad schematic)
At the start: 37 parts, among them J1 DevKitC-1 LEFT 1x22, J10 ESC_RR, J11 ESC_RL, J12 OPTIONAL 3V3 UART, J13 F2 MINI: VCC TBD, J14 0-2.5V current input, J2 DevKitC-1 RIGHT 1x22, J3 REGULATED 5V ONLY, J4 MPU6050, J5 BMP280, J6 HMC5883L, J7 SENSE ONLY, J8 ESC_FL, J9 ESC_FR

Commit message: Unify ESP32 firmware, verify optional ROS2 fallback and connect DevKit grounds directly
Parts:
- removed W22: INSULATED_WIRE, HomeEtch:W22, symbol HomeEtch:Block_2
Connections:
- net GND_MCU is gone; now on net GND: J1.22
- net GND: now also J2.1, J2.21, J2.22
- no-connect marks 30 -> 27

Commit message: Use solid common-ground pads and verify PCB power rails and toner mask
Parts:
- added W23: INSULATED_WIRE, HomeEtch:W23, symbol HomeEtch:Block_2
- J13: value F2 MINI: VCC TBD -> F2 MINI: REG 5V
Connections:
- net 3V3: now also J1.2
- net 5V_EXT: now also W23.1
- net LIDAR_5V: now reaches J13.2
- net LIDAR_5V: now also W23.2
- no-connect marks 27 -> 25

Commit message: Verify PCB reference dimensions and regenerate three actual-size copper masks
Parts:
- C1, C2: value 100nF -> 100nF X7R 5mm
- J4: value MPU6050 -> MPU6050 WIRE PORT
- J5: value BMP280 -> BMP280 WIRE PORT
- J6: value HMC5883L -> HMC5883L WIRE PORT

Commit message: Fix photo-matched sensor headers and verify single-sided PCB mask
Parts:
- added W24: INSULATED_WIRE, HomeEtch:W24, symbol HomeEtch:Block_2
- J13: value F2 MINI: REG 5V -> F2 MINI WIRE PADS
- J4: value MPU6050 WIRE PORT -> GY-521 MPU6050; symbol HomeEtch:Block_4 -> HomeEtch:Block_8
- J5: value BMP280 WIRE PORT -> GY-BM280 I2C; symbol HomeEtch:Block_4 -> HomeEtch:Block_6
- J6: value HMC5883L WIRE PORT -> GY-271 MAG; symbol HomeEtch:Block_4 -> HomeEtch:Block_5
Connections:
- net GND: now also J4.2, J4.7, J5.2, J5.6, J6.2; no longer J4.1, J5.1, J6.1
- net I2C_SCL: now also J4.3, J5.3, J6.3; no longer J4.4, J5.4, J6.4
- net I2C_SDA: now also J4.4, J5.4, J6.4; no longer J4.3, J5.3, J6.3
- net SENS_3V3: now also J4.1, J5.1, J6.1, W24.1; no longer J4.2, J5.2, J6.2
- new net BARO_CSB: J5.5, W24.2
- no-connect marks 25 -> 29
Other:
- moved on the sheet: C1, C2, J10, J11, J12, J13, J14, J7, J8, J9, R1, R2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
