File: hardware/home-etched-v3/dedicated-ground-jumpers/QCopter.kicad_sch (KiCad schematic)
At the start: 12 parts, among them J1 LIDAR_SOLDER_WIRES, J2 ESC_Servo_1x03, J3 ESC_Servo_1x03, J4 ESC_Servo_1x03, J5 ESC_Servo_1x03, U1 ESP32_S3_DevKitC_1_44pin, U2 MPU6050_GY521_1x08, U3 BMP280_GY_1x06, U4 Magnetometer_GY271_1x05

Commit message: Clear antenna-edge copper and preserve common ground with three wire links
Connections:
- net GND: no longer G1.2 (COMMON_GND), J2.1 (GND), U1.44 (GND), U3.6 (SDO)
- new net GND_RF_RETURN: G1.2 (COMMON_GND), G2.3 (RF_GND_RETURN), J2.1 (GND), U1.44 (GND), U3.6 (SDO)
